File: midi/midi.kicad_sch (KiCad schematic)
At the start: 0 parts

Commit message: did a lot
Parts:
- added D1, D2, D3, D4: SK6812MINI, LED_SMD:LED_SK6812MINI_PLCC4_3.5x3.5mm_P1.75mm, symbol LED:SK6812MINI
- added J1: Conn_01x07_Pin, capacitative keys:EXISTS, symbol Connector:Conn_01x07_Pin
- added RV1: R_Potentiometer_MountingPin, Potentiometer_THT:Potentiometer_Bourns_PTA1543_Single_Slide, symbol Device:R_Potentiometer_MountingPin
- added SW1, SW2, SW3: SW_Push, Hackclub Footprints:Kailh Choc Low-Profile Switches, symbol Switch:SW_Push
- added SW4: RotaryEncoder_Switch_MP, Rotary_Encoder:RotaryEncoder_Alps_EC11E-Switch_Vertical_H20mm, symbol Device:RotaryEncoder_Switch_MP
- added U1: Waveshare ESP32-S3-ZERO, Hackclub Footprints:Waveshare ESP32-S3-Zero, symbol Hackclub Symbols:Waveshare ESP32-S3-ZERO
Connections:
- new net: D3.2 (VSS), D4.4 (VDD)
- new net: D2.2 (VSS), D3.4 (VDD)
- new net: D1.2 (VSS), D2.4 (VDD)
- new net +3V3: D1.3 (DIN), D2.3 (DIN), D3.3 (DIN), D4.3 (DIN), U1.3V3 (3V3(OUT))
- new net +5V: U1.5V
- new net ENC1_A: SW4.A, U1.8 (GP8)
- new net ENC1_B: SW4.B, U1.9 (GP9)
- new net ENC1_SW: U1.10 (GP10)
- new net ENC_SW: SW4.S1
- new net GND: D1.1 (DOUT), D2.1 (DOUT), D3.1 (DOUT), D4.1 (DOUT), RV1.3, RV1.MP (MountPin), SW1.1, SW2.1, SW3.1, SW4.C, SW4.MP, U1.GND
- new net LED: D4.2 (VSS), U1.12 (GP12)
- new net SLIDE: RV1.2, U1.11 (GP11)
- new net SWITCH1: SW1.2, U1.RX
- new net SWITCH2: SW2.2, U1.TX
- new net SWITCH3: SW3.2, U1.13 (GP13)
- new net TOUCH1: J1.1 (Pin_1), U1.1 (GP1)
- new net TOUCH2: J1.2 (Pin_2), U1.2 (GP2)
- new net TOUCH3: J1.3 (Pin_3), U1.3 (GP3)
- new net TOUCH4: J1.4 (Pin_4), U1.4 (GP4)
- new net TOUCH5: J1.5 (Pin_5), U1.5 (GP5)
- new net TOUCH6: J1.6 (Pin_6), U1.6 (GP6)
- new net TOUCH7: J1.7 (Pin_7), U1.7 (GP7)
- no-connect marks 0 -> 2

Commit message: added screen footprinnts
Connections:
- net ENC1_A: now also U1.2 (GP2); no longer U1.8 (GP8)
- net ENC1_B: now also U1.RX; no longer U1.9 (GP9)
- net ENC1_SW: now also U1.TX; no longer U1.10 (GP10)
- net LED: now also U1.13 (GP13); no longer U1.12 (GP12)
- net SLIDE: now also U1.1 (GP1); no longer U1.11 (GP11)
- net SWITCH1: now also U1.3 (GP3); no longer U1.RX
- net SWITCH2: now also U1.4 (GP4); no longer U1.TX
- net SWITCH3: now also U1.5 (GP5); no longer U1.13 (GP13)
- net TOUCH1: now also U1.6 (GP6); no longer U1.1 (GP1)
- net TOUCH2: now also U1.7 (GP7); no longer U1.2 (GP2)
- net TOUCH3: now also U1.8 (GP8); no longer U1.3 (GP3)
- net TOUCH4: now also U1.9 (GP9); no longer U1.4 (GP4)
- net TOUCH5: now also U1.10 (GP10); no longer U1.5 (GP5)
- net TOUCH6: now also U1.11 (GP11); no longer U1.6 (GP6)
- net TOUCH7: now also U1.12 (GP12); no longer U1.7 (GP7)
